File: onlab.kicad_sch (KiCad schematic)
At the start: 82 parts, among them J1 Battery, J10 DC-Motor, J2 HC_SR04, J3 HC_SR04, J4 HC_SR04, J5 DC-Motor, J6 DC-Motor, J7 DC-Motor, J8 DC-Motor, J9 DC-Motor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

Commit message: layout v2
Connections:
- net at R12.1, SW3.3: now also U4.10 (P5); no longer U4.12 (P7)
- net at R10.1, SW3.1: now also U4.12 (P7); no longer U4.10 (P5)
Other:
- moved on the sheet: D5
Changed lines of the file:
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@@
   (junction (at 102.87 25.4) (diameter 0) (color 0 0 0 0)
   )
+  (junction (at 80.518 146.558) (diameter 0) (color 0 0 0 0)
+  )
   (junction (at 62.738 123.19) (diameter 0) (color 0 0 0 0)
   )
@@
   (junction (at 217.17 129.54) (diameter 0) (color 0 0 0 0)
   )
-  (junction (at 80.518 146.558) (diameter 0) (color 0 0 0 0)
-  )
   (junction (at 366.395 138.43) (diameter 0) (color 0 0 0 0)
   )
@@
   (junction (at 99.06 40.64) (diameter 0) (color 0 0 0 0)
   )
+  (junction (at 94.488 151.638) (diameter 0) (color 0 0 0 0)
+  )
   (junction (at 363.22 232.41) (diameter 0) (color 0 0 0 0)
   )
@@
   (junction (at 219.075 238.125) (diameter 0) (color 0 0 0 0)
   )
-  (junction (at 94.488 151.638) (diameter 0) (color 0 0 0 0)
-  )
   (junction (at 364.49 184.15) (diameter 0) (color 0 0 0 0)
   )
@@
     (stroke (width 0) (type default))
   )
-  (wire (pts (xy 94.488 151.638) (xy 97.028 151.638))
-    (stroke (width 0) (type default))
-  )
   (wire (pts (xy 190.5 59.69) (xy 193.04 59.69))
     (stroke (width 0) (type default))
@@
     (stroke (width 0) (type default))
   )
+  (wire (pts (xy 76.962 150.876) (xy 91.948 150.876))
+    (stroke (width 0) (type default))
+  )
   (wire (pts (xy 352.425 234.95) (xy 365.76 234.95))
     (stroke (width 0) (type default))
@@
     (stroke (width 0) (type default))
   )
+  (wire (pts (xy 78.486 151.638) (xy 78.486 146.558))
+    (stroke (width 0) (type default))
+  )
   (wire (pts (xy 233.045 248.92) (xy 237.49 248.92))
     (stroke (width 0) (type default))
@@
     (stroke (width 0) (type default))
   )
-  (wire (pts (xy 75.438 146.558) (xy 80.518 146.558))
-    (stroke (width 0) (type default))
-  )
   (wire (pts (xy 62.992 175.514) (xy 62.992 177.8))
     (stroke (width 0) (type default))
@@
     (stroke (width 0) (type default))
   )
+  (wire (pts (xy 91.948 151.638) (xy 94.488 151.638))
+    (stroke (width 0) (type default))
+  )
   (wire (pts (xy 88.9 40.64) (xy 92.456 40.64))
     (stroke (width 0) (type default))
   )
+  (wire (pts (xy 76.962 146.558) (xy 76.962 150.876))
+    (stroke (width 0) (type default))
+  )
   (wire (pts (xy 153.67 238.76) (xy 153.67 240.665))
     (stroke (width 0) (type default))
@@
     (stroke (width 0) (type default))
   )
+  (wire (pts (xy 94.488 151.638) (xy 97.028 151.638))
+    (stroke (width 0) (type default))
+  )
   (wire (pts (xy 337.312 38.354) (xy 339.852 38.354))
     (stroke (width 0) (type default))
@@
     (stroke (width 0) (type default))
   )
+  (wire (pts (xy 91.948 150.876) (xy 91.948 151.638))
+    (stroke (width 0) (type default))
+  )
   (wire (pts (xy 101.346 84.836) (xy 106.426 84.836))
     (stroke (width 0) (type default))
@@
     (stroke (width 0) (type default))
   )
-  (wire (pts (xy 181.102 178.054) (xy 182.372 178.054))
+  (wire (pts (xy 181.102 178.054) (xy 183.134 178.054))
     (stroke (width 0) (type default))
   )
@@
     (stroke (width 0) (type default))
   )
+  (wire (pts (xy 75.438 151.638) (xy 78.486 151.638))
+    (stroke (width 0) (type default))
+  )
   (wire (pts (xy 75.438 149.098) (xy 88.138 149.098))
     (stroke (width 0) (type default))
@@
     (stroke (width 0) (type default))
   )
+  (wire (pts (xy 75.438 146.558) (xy 76.962 146.558))
+    (stroke (width 0) (type default))
+  )
   (wire (pts (xy 276.86 129.54) (xy 273.05 129.54))
     (stroke (width 0) (type default))
@@
     (stroke (width 0) (type default))
   )
+  (wire (pts (xy 78.486 146.558) (xy 80.518 146.558))
+    (stroke (width 0) (type default))
+  )
   (wire (pts (xy 190.5 44.45) (xy 193.04 44.45))
     (stroke (width 0) (type default))
@@
     (stroke (width 0) (type default))
   )
-  (wire (pts (xy 189.992 178.054) (xy 191.262 178.054))
+  (wire (pts (xy 190.754 178.054) (xy 191.262 178.054))
     (stroke (width 0) (type default))
   )
@@
     (stroke (width 0) (type default))
   )
-  (wire (pts (xy 75.438 151.638) (xy 94.488 151.638))
-    (stroke (width 0) (type default))
-  )
   (wire (pts (xy 337.185 135.89) (xy 363.22 135.89))
     (stroke (width 0) (type default))
@@
     )
   )
+  (netclass_flag "" (length 2.54) (shape round) (at 266.954 68.326 270) (fields_autoplaced)
+    (effects (font (size 1.27 1.27)) (justify right bottom))
+    (property "Netclass" "signal" (at 269.494 69.0245 90)
+      (effects (font (size 1.27 1.27) italic) (justify right))
+    )
+  )
   (netclass_flag "" (length 2.54) (shape round) (at 150.114 248.92 180) (fields_autoplaced)
     (effects (font (size 1.27 1.27)) (justify right bottom))
@@
     )
   )
-  (netclass_flag "" (length 2.54) (shape round) (at 86.614 148.844 0) (fields_autoplaced)
+  (netclass_flag "" (length 2.54) (shape round) (at 86.614 149.098 0) (fields_autoplaced)
     (effects (font (size 1.27 1.27)) (justify left bottom))
-    (property "Netclass" "signal" (at 87.3125 146.304 0)
+    (property "Netclass" "signal" (at 87.3125 146.558 0)
       (effects (font (size 1.27 1.27) italic) (justify left))
     )
@@
     )
   )
+  (netclass_flag "" (length 2.54) (shape round) (at 178.308 39.37 0) (fields_autoplaced)
+    (effects (font (size 1.27 1.27)) (justify left bottom))
+    (property "Netclass" "signal" (at 179.0065 36.83 0)
+      (effects (font (size 1.27 1.27) italic) (justify left))
+    )
+  )
+  (netclass_flag "" (length 2.54) (shape round) (at 370.84 70.104 0) (fields_autoplaced)
+    (effects (font (size 1.27 1.27)) (justify left bottom))
+    (property "Netclass" "signal" (at 371.5385 67.564 0)
+      (effects (font (size 1.27 1.27) italic) (justify left))
+    )
+  )
   (netclass_flag "" (length 2.54) (shape round) (at 78.994 23.368 90) (fields_autoplaced)
     (effects (font (size 1.27 1.27)) (justify left bottom))
@@
     )
   )
+  (netclass_flag "" (length 2.54) (shape round) (at 370.586 39.624 0) (fields_autoplaced)
+    (effects (font (size 1.27 1.27)) (justify left bottom))
+    (property "Netclass" "signal" (at 371.2845 37.084 0)
+      (effects (font (size 1.27 1.27) italic) (justify left))
+    )
+  )
   (symbol (lib_id "power:VCC") (at 335.534 77.724 0) (unit 1)
     (in_bom yes) (on_board yes) (dnp no)
@@
     )
   )
-  (symbol (lib_id "Device:LED") (at 186.182 178.054 0) (unit 1)
+  (symbol (lib_id "Device:LED") (at 186.944 178.054 0) (unit 1)
     (in_bom yes) (on_board yes) (dnp no)
-    (property "Reference" "D5" (at 186.182 180.594 0)
+    (property "Reference" "D5" (at 186.944 180.594 0)
       (effects (font (size 1.27 1.27)))
     )
-    (property "Value" "LED" (at 186.182 175.514 0)
+    (property "Value" "LED" (at 186.944 175.514 0)
       (effects (font (size 1.27 1.27)))
     )
-    (property "Footprint" "LED_SMD:LED_0805_2012Metric_Pad1.15x1.40mm_HandSolder" (at 186.182 178.054 0)
+    (property "Footprint" "LED_SMD:LED_0805_2012Metric_Pad1.15x1.40mm_HandSolder" (at 186.944 178.054 0)
       (effects (font (size 1.27 1.27)) hide)
     )
-    (property "Datasheet" "~" (at 186.182 178.054 0)
+    (property "Datasheet" "~" (at 186.944 178.054 0)
       (effects (font (size 1.27 1.27)) hide)
     )
