File: onlab.kicad_pcb (KiCad board)
At the start: 2 copper layers, 100 x 100 mm, 87 parts, among them J1 Battery, J10 DC-Motor, J2 HC_SR04, J3 HC_SR04, J4 HC_SR04, J5 DC-Motor, J6 DC-Motor, J7 DC-Motor, J8 DC-Motor, J9 DC-Motor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

Commit message: keep out area update, pdf update
Routing:
- net /Mot2_EncA: track 118.9 -> 119.7 mm
- net GND: vias 8 -> 7
